File: macro33.kicad_pcb (KiCad board)
At the start: 2 copper layers, 9 parts, among them SW1 SW_Push, SW2 SW_Push, SW3 SW_Push, SW4 SW_Push, SW5 SW_Push, SW6 SW_Push, SW7 SW_Push, SW8 SW_Push, SW9 SW_Push

Commit message: feat: finished design
Parts:
- added C1: 12pF, Capacitor_SMD:C_0402_1005Metric, F.Cu at (54.5, 67.8)
- added C10: 100nF, Capacitor_SMD:C_0402_1005Metric, F.Cu at (71.5, 71.2)
- added C11: 100nF, Capacitor_SMD:C_0402_1005Metric, F.Cu at (64.2, 76.2)
- added C12: 100nF, Capacitor_SMD:C_0402_1005Metric, F.Cu at (64.0, 64.0)
- added C13: 100nF, Capacitor_SMD:C_0402_1005Metric, F.Cu at (70.5, 76.2)
- added C14: 10uF, Capacitor_SMD:C_1206_3216Metric, F.Cu at (90.8, 68.5)
- added C15: 10uF, Capacitor_SMD:C_1206_3216Metric, F.Cu at (99.5, 61.5)
- added C16: 100nf, Capacitor_SMD:C_0402_1005Metric, F.Cu at (70.5, 75.2)
- added C2: 12pF, Capacitor_SMD:C_0402_1005Metric, F.Cu at (56.0, 73.8)
- added C3: 100nF, Capacitor_SMD:C_0402_1005Metric, F.Cu at (58.5, 73.8)
- added C4: 1uF, Capacitor_SMD:C_0402_1005Metric, F.Cu at (70.5, 74.2)
- added C5: 100nF, Capacitor_SMD:C_0402_1005Metric, F.Cu at (72.5, 69.8)
- added C6: 1uF, Capacitor_SMD:C_0402_1005Metric, F.Cu at (70.5, 77.2)
- added C7: 100nF, Capacitor_SMD:C_0402_1005Metric, F.Cu at (69.0, 65.8)
- added C8: 100nF, Capacitor_SMD:C_0402_1005Metric, F.Cu at (104.0, 74.0)
- added C9: 100nF, Capacitor_SMD:C_0402_1005Metric, F.Cu at (58.5, 71.8)
- added JP1: SolderJumper_2_Open, Jumper:SolderJumper-2_P1.3mm_Open_TrianglePad1.0x1.5mm, F.Cu at (105.2, 70.0)
- added R1: 27r, Resistor_SMD:R_0805_2012Metric, F.Cu at (74.5, 71.8)
- added R2: 27r, Resistor_SMD:R_0805_2012Metric, F.Cu at (74.6, 73.8)
- added R3: 1k, Resistor_SMD:R_0402_1005Metric, F.Cu at (104.0, 67.5)
- added R5: 5.1k, Resistor_SMD:R_0402_1005Metric, F.Cu at (84.0, 71.6)
- added SWD: Conn_01x03_Socket, Library:SWD-Pads, F.Cu at (58.8, 78.9)
- added U1: RP2040, Package_DFN_QFN:QFN-56-1EP_7x7mm_P0.4mm_EP3.2x3.2mm, F.Cu at (65.2, 71.2)
- added U2: W25Q128JVS, Package_SO:SOIC-8_5.23x5.23mm_P1.27mm, F.Cu at (100.5, 71.0)
- added U3: NCP1117-3.3_SOT223, Package_TO_SOT_SMD:SOT-223-3_TabPin2, F.Cu at (92.8, 63.8)
- added USBC1: ~, Library:USB-C-SMD_C67380, F.Cu at (81.8, 64.4)
- added Y1: XYDBPCNANF-12MHZ, Library:OSC-SMD_4P-L2.5-W2.0-BL, F.Cu at (55.2, 70.8)
- SW1, SW2, SW3, SW4, SW5, SW6, SW7, SW8, SW9: moved to B.Cu
- moved SW3 67.4 mm to (100.8, 85.8)
- moved SW2 63.9 mm to (81.8, 85.8)
- moved SW6 63.9 mm to (100.8, 104.8)
- moved SW1 60.7 mm to (62.8, 85.8)
- moved SW9 60.7 mm to (100.8, 123.8)
- moved SW5 60.3 mm to (81.8, 104.8)
- moved SW4 56.9 mm to (62.8, 104.8)
- moved SW8 56.8 mm to (81.8, 123.8)
- moved SW7 53.2 mm to (62.8, 123.8)
Connections:
- SW1 pad 1: unconnected-(SW1-Pad1) -> /GPIO_8
- SW1 pad 2: unconnected-(SW1-Pad2) -> GND
- SW2 pad 1: unconnected-(SW2-Pad1) -> /GPIO_3
- SW2 pad 2: unconnected-(SW2-Pad2) -> GND
- SW3 pad 1: unconnected-(SW3-Pad1) -> /GPIO_0
- SW3 pad 2: unconnected-(SW3-Pad2) -> GND
- SW4 pad 1: unconnected-(SW4-Pad1) -> /GPIO_7
- SW4 pad 2: unconnected-(SW4-Pad2) -> GND
- SW5 pad 1: unconnected-(SW5-Pad1) -> /GPIO_4
- SW5 pad 2: unconnected-(SW5-Pad2) -> GND
- SW6 pad 1: unconnected-(SW6-Pad1) -> /GPIO_1
- SW6 pad 2: unconnected-(SW6-Pad2) -> GND
- SW7 pad 1: unconnected-(SW7-Pad1) -> /GPIO_6
- SW7 pad 2: unconnected-(SW7-Pad2) -> GND
- SW8 pad 1: unconnected-(SW8-Pad1) -> /GPIO_5
- SW8 pad 2: unconnected-(SW8-Pad2) -> GND
- SW9 pad 1: unconnected-(SW9-Pad1) -> /GPIO_2
- SW9 pad 2: unconnected-(SW9-Pad2) -> GND
Routing:
- net /GPIO_2: track 0.00 -> 85.1 mm, vias 0 -> 1
- net GND: track 0.00 -> 81.9 mm, vias 0 -> 28
- net /GPIO_6: track 0.00 -> 80.1 mm, vias 0 -> 1
- net /GPIO_5: track 0.00 -> 70.6 mm, vias 0 -> 1
- net /GPIO_1: track 0.00 -> 66.4 mm, vias 0 -> 1
- net /GPIO_7: track 0.00 -> 59.7 mm, vias 0 -> 1
- net /GPIO_4: track 0.00 -> 51.4 mm, vias 0 -> 1
- net /GPIO_0: track 0.00 -> 45.4 mm, vias 0 -> 1
- net /QSPI_SS: track 0.00 -> 44.6 mm, vias 0 -> 2
- net /QSPI_SD1: track 0.00 -> 42.2 mm, vias 0 -> 2
- net /QSPI_SD2: track 0.00 -> 41.3 mm, vias 0 -> 2
- net /QSPI_SD3: track 0.00 -> 38.9 mm, vias 0 -> 2
- net /QSPI_SCLK: track 0.00 -> 38.5 mm, vias 0 -> 2
- net /QSPI_SD0: track 0.00 -> 36.6 mm, vias 0 -> 2
- net VBUS: track 0.00 -> 33.0 mm
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- added copper zone on F.Cu, net +1V1
- added copper zone on F.Cu, net +3.3V
- added copper zone on B.Cu, net GND
- added copper zone on F.Cu, net VBUS
Other:
- board outline added: 56.5 x 73.2 mm
- board text added: "https://github.com/GameTec-live/macro33"

Commit message: feat: rev2
Parts:
- C16: value 100nf -> 100nF
- moved C1 53.9 mm to (108.0, 73.9), turned to 90 degrees
- moved Y1 52.0 mm to (107.2, 70.8), turned to -90 degrees
- moved C2 50.8 mm to (106.5, 67.9), turned to -90 degrees
- moved C9 46.2 mm to (104.5, 67.8), turned to 90 degrees
- moved C3 45.4 mm to (103.5, 67.9), turned to 90 degrees
- moved C8 42.8 mm to (61.2, 73.5)
- moved R3 42.8 mm to (61.2, 67.0)
- moved U2 42.8 mm to (57.8, 70.5)
- moved RST 42.8 mm to (62.5, 69.5)
- moved C12 37.9 mm to (100.0, 75.6), turned to 0 degrees
- moved C11 37.0 mm to (99.8, 65.8), turned to 0 degrees
- moved C15 35.2 mm to (65.5, 70.4), turned to -90 degrees
- moved U1 33.0 mm to (98.2, 70.5), turned to 90 degrees
- moved C7 27.5 mm to (94.9, 75.1), turned to 180 degrees
- moved C6 27.1 mm to (95.0, 65.8)
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- renumbered JP1 to RST
Connections:
- SW1 pad 1: /GPIO_8 -> /GPIO_0
- SW3 pad 1: /GPIO_0 -> /GPIO_6
- SW4 pad 1: /GPIO_7 -> /GPIO_1
- SW6 pad 1: /GPIO_1 -> /GPIO_7
- SW7 pad 1: /GPIO_6 -> /GPIO_2
- SW9 pad 1: /GPIO_2 -> /GPIO_8
- U1 pad 26: /RUN -> unconnected-(U1-RUN-Pad26)
Routing:
- net +3.3V: track 28.9 -> 103.4 mm, vias 0 -> 6
- net /GPIO_6: track 80.1 -> 19.2 mm, vias 1 -> 0
- net /SWCLK: track 8.12 -> 66.5 mm, vias 0 -> 2
- net /SWD: track 5.42 -> 59.0 mm, vias 0 -> 2
- net /GPIO_8: track 28.2 -> 72.9 mm, vias 1 -> 0
- net GND: track 81.9 -> 56.6 mm, vias 28 -> 34
- net /GPIO_0: track 45.4 -> 69.3 mm, vias 1 -> 0
- net /GPIO_3: track 31.0 -> 52.2 mm, vias 1 -> 0
- net /QSPI_SS: track 44.6 -> 59.0 mm
- net /QSPI_SD1: track 42.2 -> 54.2 mm
- net /QSPI_SD2: track 41.3 -> 51.2 mm
- net /QSPI_SD0: track 36.6 -> 45.7 mm
- net VBUS: track 33.0 -> 27.0 mm
- net /QSPI_SCLK: track 38.5 -> 44.4 mm
- net /D-: track 18.5 -> 24.2 mm
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- added copper zone on F.Cu, net GND
- removed copper zone on F.Cu, net +3.3V
Other:
- board size 56.5 x 73.2 mm -> 56.5 x 68.5 mm
