File: macro33.kicad_sch (KiCad schematic)
At the start: 9 parts, among them SW1 SW_Push, SW2 SW_Push, SW3 SW_Push, SW4 SW_Push, SW5 SW_Push, SW6 SW_Push, SW7 SW_Push, SW8 SW_Push, SW9 SW_Push

Commit message: feat: finished design
Parts:
- added C1, C2: 12pF, Capacitor_SMD:C_0402_1005Metric, symbol Device:C
- added C10, C11, C12, C13, C3, C5, C7, C8, C9: 100nF, Capacitor_SMD:C_0402_1005Metric, symbol Device:C
- added C14, C15: 10uF, Capacitor_SMD:C_1206_3216Metric, symbol Device:C
- added C16: 100nf, Capacitor_SMD:C_0402_1005Metric, symbol Device:C
- added C4, C6: 1uF, Capacitor_SMD:C_0402_1005Metric, symbol Device:C
- added J1: Conn_01x03_Socket, Library:SWD-Pads, symbol Connector:Conn_01x03_Socket
- added JP1: SolderJumper_2_Open, Jumper:SolderJumper-2_P1.3mm_Open_TrianglePad1.0x1.5mm, symbol Jumper:SolderJumper_2_Open
- added R1, R2: 27r, Resistor_SMD:R_0805_2012Metric, symbol Device:R
- added R3: 1k, Resistor_SMD:R_0402_1005Metric, symbol Device:R
- added R5: 5.1k, Resistor_SMD:R_0402_1005Metric, symbol Device:R
- added U1: RP2040, Package_DFN_QFN:QFN-56-1EP_7x7mm_P0.4mm_EP3.2x3.2mm, symbol MCU_RaspberryPi:RP2040
- added U2: W25Q128JVS, Package_SO:SOIC-8_5.23x5.23mm_P1.27mm, symbol Memory_Flash:W25Q128JVS
- added U3: NCP1117-3.3_SOT223, Package_TO_SOT_SMD:SOT-223-3_TabPin2, symbol Regulator_Linear:NCP1117-3.3_SOT223
- added USBC1: ~, Library:USB-C-SMD_C67380, symbol Library:FUC-24F11-SNLB1
- added Y1: XYDBPCNANF-12MHZ, Library:OSC-SMD_4P-L2.5-W2.0-BL, symbol Device:Crystal_GND24
Connections:
- net GPIO_0: now reaches SW3.1
- net GPIO_0: now also U1.2 (GPIO0)
- net GND: now reaches SW3.2
- net GND: now also SW1.2, SW2.2, SW4.2, SW5.2, SW6.2, SW7.2, SW8.2, SW9.2, C1.1, C10.2, C11.2, C12.2, C13.2, C14.2, C15.2, C16.2, C2.1, C3.2, C4.2, C5.2, C6.2, C7.2, C8.2, C9.2, J1.3 (Pin_3), JP1.1 (A), R5.1, U1.19 (TESTEN), U1.57 (GND), U2.4 (GND), U3.1 (GND), USBC1.A1 (GND), USBC1.A12 (GND), USBC1.B1 (GND), USBC1.B12 (GND), Y1.2, Y1.4
- net GPIO_8: now reaches SW1.1
- net GPIO_8: now also U1.11 (GPIO8)
- net GPIO_6: now reaches SW7.1
- net GPIO_6: now also U1.8 (GPIO6)
- net GPIO_3: now reaches SW2.1
- net GPIO_3: now also U1.5 (GPIO3)
- net GPIO_4: now reaches SW5.1
- net GPIO_4: now also U1.6 (GPIO4)
- net GPIO_5: now reaches SW8.1
- net GPIO_5: now also U1.7 (GPIO5)
- net GPIO_1: now reaches SW6.1
- net GPIO_1: now also U1.3 (GPIO1)
- net GPIO_2: now reaches SW9.1
- net GPIO_2: now also U1.4 (GPIO2)
- net GPIO_7: now reaches SW4.1
- net GPIO_7: now also U1.9 (GPIO7)
- new net: C1.2, U1.20 (XIN), Y1.3
- new net: C2.2, U1.21 (XOUT), Y1.1
- new net: R2.2, U1.46 (USB_DM)
- new net: R1.2, U1.47 (USB_DP)
- new net: JP1.2 (B), R3.1
- new net: R5.2, USBC1.A5 (CC1), USBC1.B5 (CC2)
- new net +1V1: C3.1, C4.1, C5.1, U1.23 (DVDD), U1.45 (VREG_VOUT), U1.50 (DVDD)
- new net +3.3V: C10.1, C11.1, C12.1, C13.1, C15.1, C16.1, C6.1, C7.1, C8.1, C9.1, U1.1 (IOVDD), U1.10 (IOVDD), U1.22 (IOVDD), U1.33 (IOVDD), U1.42 (IOVDD), U1.43 (ADC_AVDD), U1.44 (VREG_IN), U1.48 (USB_VDD), U1.49 (IOVDD), U2.8 (VCC), U3.2 (VO)
- new net D+: R1.1, USBC1.A6 (DP1), USBC1.B6 (DP2)
- new net D-: R2.1, USBC1.A7 (DN1), USBC1.B7 (DN2)
- new net QSPI_SCLK: U1.52 (QSPI_SCLK), U2.6 (CLK)
- new net QSPI_SD0: U1.53 (QSPI_SD0), U2.5 (DI(IO0))
- new net QSPI_SD1: U1.55 (QSPI_SD1), U2.2 (DO(IO1))
- new net QSPI_SD2: U1.54 (QSPI_SD2), U2.3 (IO2)
- new net QSPI_SD3: U1.51 (QSPI_SD3), U2.7 (IO3)
- new net QSPI_SS: R3.2, U1.56 (QSPI_SS), U2.1 (~{CS})
- new net RUN: U1.26 (RUN)
- new net SWCLK: J1.1 (Pin_1), U1.24 (SWCLK)
- new net SWD: J1.2 (Pin_2), U1.25 (SWD)
- new net VBUS: C14.1, U3.3 (VI), USBC1.A4 (VBUS), USBC1.A9 (VBUS), USBC1.B4 (VBUS), USBC1.B9 (VBUS)
- no-connect marks 0 -> 35
Other:
- note added: "boot select"
- note added: "place close to pin 44"
- note added: "place close to pin 45"
- title: (none) -> Macro33
- moved on the sheet: SW1, SW2, SW3, SW4, SW5, SW6, SW7, SW8, SW9

Commit message: feat: gerbers
Parts:
- C16: value 100nf -> 100nF
Changed lines of the file:
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@@
 			)
 		)
-		(property "Value" "100nf"
+		(property "Value" "100nF"
 			(at 91.44 153.6699 0)
 			(effects

Commit message: feat: rev2
Connections:
- net GPIO_0: now also SW1.1; no longer SW3.1
- net GPIO_1: now also SW4.1; no longer SW6.1
- net GPIO_2: now also SW7.1; no longer SW9.1
- net GPIO_6: now also SW3.1; no longer SW7.1
- net GPIO_7: now also SW6.1; no longer SW4.1
- net GPIO_8: now also SW9.1; no longer SW1.1
- net RUN: no longer names the net of U1.26 (RUN)
- no-connect marks 35 -> 36
Changed lines of the file:
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@@
 		(title "Macro33")
 		(date "2025-02-10")
-		(rev "1")
+		(rev "2")
 		(comment 1 "GPLV3 Licensed")
 	)
@@
 	)
 	(no_connect
+		(at 147.32 78.74)
+	)
+	(no_connect
 		(at 198.12 134.62)
 	)
@@
 		(pts
 			(xy 143.51 109.22) (xy 147.32 109.22)
-		)
-		(stroke
-			(width 0)
-			(type default)
-		)
-	)
-	(wire
-		(pts
-			(xy 146.05 78.74) (xy 147.32 78.74)
 		)
 		(stroke
@@
 		)
 	)
+	(label "GPIO_1"
+		(at 214.63 99.06 180)
+		(effects
+			(font
+				(size 1 1)
+			)
+			(justify right bottom)
+		)
+	)
 	(label "D+"
 		(at 95.25 71.12 0)
@@
 	)
 	(label "GPIO_7"
-		(at 214.63 99.06 180)
+		(at 265.43 99.06 180)
+		(effects
+			(font
+				(size 1 1)
+			)
+			(justify right bottom)
+		)
+	)
+	(label "GPIO_0"
+		(at 214.63 86.36 180)
 		(effects
 			(font
@@
 		)
 	)
-	(label "GPIO_2"
-		(at 265.43 111.76 180)
-		(effects
-			(font
-				(size 1 1)
-			)
-			(justify right bottom)
-		)
-	)
 	(label "GPIO_0"
 		(at 201.93 78.74 0)
@@
 		)
 	)
+	(label "GPIO_2"
+		(at 214.63 111.76 180)
+		(effects
+			(font
+				(size 1 1)
+			)
+			(justify right bottom)
+		)
+	)
 	(label "GPIO_8"
 		(at 201.93 99.06 0)
@@
 		)
 	)
-	(label "GPIO_6"
-		(at 214.63 111.76 180)
-		(effects
-			(font
-				(size 1 1)
-			)
-			(justify right bottom)
-		)
-	)
 	(label "GPIO_1"
 		(at 201.93 81.28 0)
@@
 		)
 	)
-	(label "RUN"
-		(at 146.05 78.74 180)
-		(effects
-			(font
-				(size 1 1)
-			)
-			(justify right bottom)
-		)
-	)
 	(label "SWD"
 		(at 250.19 121.92 180)
@@
 		)
 	)
-	(label "GPIO_1"
-		(at 265.43 99.06 180)
+	(label "GPIO_8"
+		(at 265.43 111.76 180)
 		(effects
 			(font
@@
 		)
 	)
-	(label "GPIO_0"
+	(label "GPIO_6"
 		(at 265.43 86.36 180)
 		(effects
 			(font
-				(size 1 1)
-			)
-			(justify right bottom)
-		)
-	)
-	(label "GPIO_8"
-		(at 214.63 86.36 180)
-		(effects
-			(font
